File: hardware/kicad/PocketMate.kicad_pcb (KiCad board)
At the start: 6 copper layers, 55 x 69.8 mm, 150 parts, among them J1 10164227-1001A1RLF, J10 Skin NTC 10k B3435, J11 FH12-16S-0.5SH(55), J12 Fan 5V/GND/PWM/TACH, J2 10164227-1001A1RLF, J3 DSI1 22p 0.5mm FH12-22S-0.5SH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, J4 CSI0 22p 0.5mm FH12-22S-0.5SH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, J5 Speaker 8R 1W, J6 TYPE-C-31-M-12, J7 Molex 205338-0005 (BAT+,BAT+,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, J8 SWD (TC2030 pads), J9 LRA motor, Q1 DMP3013SFV, Q2 DMP3013SFV, Q3 2N7002, Q4 2N7002, Q5 2N7002, Q6 2N7002, U1 MAX98357AETE+, U11 DRV2605LDGSR, U12 TLV62585DRLR, U13 TPD4E05U06DQAR (flex buttons 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, U14 TPS22917DBVR, U2 USBLC6-2SC6 (D+/D-), U3 USBLC6-2SC6 (CC1/CC2), U4 STUSB4500QTR, U5 BQ25895RTWR, U6 MAX17055ETB+, U7 TPS7A0233PDBVR, U8 TPS61088RHLR, U9 STM32U031K8U6

Commit message: Sync PCB layout and design rules with latest source
Parts:
- added C61: 22uF, Capacitor_SMD:C_0805_2012Metric, F.Cu at (8.08, 4.04)
- added C62: 100nF, Capacitor_SMD:C_0402_1005Metric, F.Cu at (8.21, 1.33)
- added J14: LTE link FH12-22S-0.5SH(55), Connector_FFC-FPC:Hirose_FH12-22S-0.5SH_1x22-1MP_P0.50mm_Horizontal, F.Cu at (4.00, 6.50)
- added R56: 0R, Resistor_SMD:R_0402_1005Metric, F.Cu at (8.21, 7.22)
- added R57: 100k, Resistor_SMD:R_0402_1005Metric, F.Cu at (8.24, 8.25)
- C25, R6: moved to F.Cu
- moved C28 42.9 mm to (24.8, -13.6), turned to 0 degrees
- moved C27 42.9 mm to (23.3, -14.9)
- moved C46 31.8 mm to (9.92, -1.77)
- moved C8 29.6 mm to (13.1, -15.2), turned to 0 degrees
- moved C44 29.1 mm to (9.24, 0.26)
- moved C45 27.5 mm to (9.77, 1.78)
- moved R23 20.8 mm to (17.8, 4.80), turned to 90 degrees
- moved R21 17.0 mm to (17.8, 2.30)
- moved C6 13.8 mm to (34.3, -1.34), turned to 0 degrees
- moved C23 11.6 mm to (20.6, -13.6), turned to 0 degrees
- moved R46 11.0 mm to (12.3, -13.6)
- moved R18 10.3 mm to (10.8, -9.48), turned to 0 degrees
- moved C24 9.97 mm to (20.4, -12.0), turned to 0 degrees
- moved R33 7.23 mm to (15.8, 15.0)
- moved C22 6.95 mm to (15.6, 17.1), turned to 0 degrees
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Connections:
- J1 pad 24: unconnected-(J1-GPIO26-Pad24) -> LTE_W_DISABLE_N
- J1 pad 28: unconnected-(J1-GPIO13-Pad28) -> LTE_RESET
- J1 pad 29: unconnected-(J1-GPIO16-Pad29) -> LTE_STATUS
- J1 pad 30: unconnected-(J1-GPIO6-Pad30) -> LTE_PWRKEY
- J1 pad 31: unconnected-(J1-GPIO12-Pad31) -> LTE_RI
- J1 pad 34: unconnected-(J1-GPIO5-Pad34) -> LTE_PWR_EN
- J1 pad 41: unconnected-(J1-GPIO25-Pad41) -> LTE_AP_READY
- J2 pad 134: unconnected-(J2-USB3-0-DP-Pad134) -> LTE_USB_DP
- J2 pad 136: unconnected-(J2-USB3-0-DM-Pad136) -> LTE_USB_DM
