File: hardware/kicad/PocketMate.kicad_sch (KiCad schematic)
At the start: 0 parts

Commit message: Sync KiCad schematic to netlist v3.2; add side_flex sheet
Other:
- added sheet SideFlex (side_flex.kicad_sch)
Changed lines of the file:
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@@
  (property "Sheetname" "CM5" (at 25.4 39.94 0) (effects (font (size 1.27 1.27)) (justify left bottom)))
  (property "Sheetfile" "cm5.kicad_sch" (at 25.4 66.64 0) (effects (font (size 1.27 1.27)) (justify left top)))
- (instances (project "PocketMate" (path "/57b5ad9e-7104-4660-a18b-c15421dfc452" (page "2")))))
+ (instances (project "PocketMate" (path "/585c1fdb-a805-5b7d-8695-92e7ad240a2e" (page "2")))))
 (sheet (at 86.36 40.64) (size 50.8 25.4) (exclude_from_sim no) (in_bom yes) (on_board yes) (dnp no) (fields_autoplaced yes) (stroke (width 0.1524) (type solid)) (fill (color 0 0 0 0))
  (property "Sheetname" "DisplayCamera" (at 86.36 39.94 0) (effects (font (size 1.27 1.27)) (justify left bottom)))
  (property "Sheetfile" "display_camera.kicad_sch" (at 86.36 66.64 0) (effects (font (size 1.27 1.27)) (justify left top)))
- (instances (project "PocketMate" (path "/57b5ad9e-7104-4660-a18b-c15421dfc452" (page "3")))))
+ (instances (project "PocketMate" (path "/585c1fdb-a805-5b7d-8695-92e7ad240a2e" (page "3")))))
 (sheet (at 147.32 40.64) (size 50.8 25.4) (exclude_from_sim no) (in_bom yes) (on_board yes) (dnp no) (fields_autoplaced yes) (stroke (width 0.1524) (type solid)) (fill (color 0 0 0 0))
  (property "Sheetname" "Audio" (at 147.32 39.94 0) (effects (font (size 1.27 1.27)) (justify left bottom)))
  (property "Sheetfile" "audio.kicad_sch" (at 147.32 66.64 0) (effects (font (size 1.27 1.27)) (justify left top)))
- (instances (project "PocketMate" (path "/57b5ad9e-7104-4660-a18b-c15421dfc452" (page "4")))))
+ (instances (project "PocketMate" (path "/585c1fdb-a805-5b7d-8695-92e7ad240a2e" (page "4")))))
 (sheet (at 208.28 40.64) (size 50.8 25.4) (exclude_from_sim no) (in_bom yes) (on_board yes) (dnp no) (fields_autoplaced yes) (stroke (width 0.1524) (type solid)) (fill (color 0 0 0 0))
  (property "Sheetname" "PowerInput" (at 208.28 39.94 0) (effects (font (size 1.27 1.27)) (justify left bottom)))
  (property "Sheetfile" "power_input.kicad_sch" (at 208.28 66.64 0) (effects (font (size 1.27 1.27)) (justify left top)))
- (instances (project "PocketMate" (path "/57b5ad9e-7104-4660-a18b-c15421dfc452" (page "5")))))
+ (instances (project "PocketMate" (path "/585c1fdb-a805-5b7d-8695-92e7ad240a2e" (page "5")))))
 (sheet (at 25.4 81.28) (size 50.8 25.4) (exclude_from_sim no) (in_bom yes) (on_board yes) (dnp no) (fields_autoplaced yes) (stroke (width 0.1524) (type solid)) (fill (color 0 0 0 0))
  (property "Sheetname" "Regulators" (at 25.4 80.58 0) (effects (font (size 1.27 1.27)) (justify left bottom)))
  (property "Sheetfile" "regulators.kicad_sch" (at 25.4 107.28 0) (effects (font (size 1.27 1.27)) (justify left top)))
- (instances (project "PocketMate" (path "/57b5ad9e-7104-4660-a18b-c15421dfc452" (page "6")))))
+ (instances (project "PocketMate" (path "/585c1fdb-a805-5b7d-8695-92e7ad240a2e" (page "6")))))
 (sheet (at 86.36 81.28) (size 50.8 25.4) (exclude_from_sim no) (in_bom yes) (on_board yes) (dnp no) (fields_autoplaced yes) (stroke (width 0.1524) (type solid)) (fill (color 0 0 0 0))
  (property "Sheetname" "MCU" (at 86.36 80.58 0) (effects (font (size 1.27 1.27)) (justify left bottom)))
  (property "Sheetfile" "mcu.kicad_sch" (at 86.36 107.28 0) (effects (font (size 1.27 1.27)) (justify left top)))
- (instances (project "PocketMate" (path "/57b5ad9e-7104-4660-a18b-c15421dfc452" (page "7")))))
+ (instances (project "PocketMate" (path "/585c1fdb-a805-5b7d-8695-92e7ad240a2e" (page "7")))))
 (sheet (at 147.32 81.28) (size 50.8 25.4) (exclude_from_sim no) (in_bom yes) (on_board yes) (dnp no) (fields_autoplaced yes) (stroke (width 0.1524) (type solid)) (fill (color 0 0 0 0))
  (property "Sheetname" "Sensors" (at 147.32 80.58 0) (effects (font (size 1.27 1.27)) (justify left bottom)))
  (property "Sheetfile" "sensors_haptics.kicad_sch" (at 147.32 107.28 0) (effects (font (size 1.27 1.27)) (justify left top)))
- (instances (project "PocketMate" (path "/57b5ad9e-7104-4660-a18b-c15421dfc452" (page "8")))))
+ (instances (project "PocketMate" (path "/585c1fdb-a805-5b7d-8695-92e7ad240a2e" (page "8")))))
+(sheet (at 208.28 81.28) (size 50.8 25.4) (exclude_from_sim no) (in_bom yes) (on_board yes) (dnp no) (fields_autoplaced yes) (stroke (width 0.1524) (type solid)) (fill (color 0 0 0 0))
+ (property "Sheetname" "SideFlex" (at 208.28 80.58 0) (effects (font (size 1.27 1.27)) (justify left bottom)))
+ (property "Sheetfile" "side_flex.kicad_sch" (at 208.28 107.28 0) (effects (font (size 1.27 1.27)) (justify left top)))
+ (instances (project "PocketMate" (path "/585c1fdb-a805-5b7d-8695-92e7ad240a2e" (page "9")))))
  (text "PocketMate CM5 carrier v0.1 - see hardware/block-diagram.md for block diagram, power tree and power states" (exclude_from_sim no) (at 25.4 25.4 0) (effects (font (size 2.54 2.54)) (justify left bottom)))
  (sheet_instances (path "/" (page "1")))

Commit message: Sync schematic with LTE link sheet (lte_link.kicad_sch), generator, nets, ERC report and PDF
Other:
- added sheet LTE (lte_link.kicad_sch)
Changed lines of the file:
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@@
  (property "Sheetfile" "side_flex.kicad_sch" (at 208.28 107.28 0) (effects (font (size 1.27 1.27)) (justify left top)))
  (instances (project "PocketMate" (path "/585c1fdb-a805-5b7d-8695-92e7ad240a2e" (page "9")))))
+(sheet (at 25.4 121.92) (size 50.8 25.4) (exclude_from_sim no) (in_bom yes) (on_board yes) (dnp no) (fields_autoplaced yes) (stroke (width 0.1524) (type solid)) (fill (color 0 0 0 0))
+ (property "Sheetname" "LTE" (at 25.4 121.22 0) (effects (font (size 1.27 1.27)) (justify left bottom)))
+ (property "Sheetfile" "lte_link.kicad_sch" (at 25.4 147.92 0) (effects (font (size 1.27 1.27)) (justify left top)))
+ (instances (project "PocketMate" (path "/585c1fdb-a805-5b7d-8695-92e7ad240a2e" (page "10")))))
  (text "PocketMate CM5 carrier v0.1 - see hardware/block-diagram.md for block diagram, power tree and power states" (exclude_from_sim no) (at 25.4 25.4 0) (effects (font (size 2.54 2.54)) (justify left bottom)))
  (sheet_instances (path "/" (page "1")))
