File: hardware/kicad/audio.kicad_sch (KiCad schematic)
At the start: 18 parts, among them J5 Speaker 8R 1W, SW1 MIC MUTE (DPDT slide), U1 MAX98357AETE+

Commit message: Sync KiCad schematic to netlist v3.2; add side_flex sheet
Parts:
- removed C11, C14: 100nF, Capacitor_SMD:C_0402_1005Metric, symbol Device:C
- removed D1: RED mic-muted, LED_SMD:LED_0402_1005Metric, symbol Device:LED
- removed MK1: SPH0645LM4H-B (Left), Sensor_Audio:Knowles_SPH0645LM4H-6_3.5x2.65mm, symbol Sensor_Audio:SPH0645LM4H
- removed MK2: SPH0645LM4H-B (Right), Sensor_Audio:Knowles_SPH0645LM4H-6_3.5x2.65mm, symbol Sensor_Audio:SPH0645LM4H
- removed R11: 100k, Resistor_SMD:R_0402_1005Metric, symbol Device:R
- removed R12: 1M, Resistor_SMD:R_0402_1005Metric, symbol Device:R
- removed R5, R6: 33R, Resistor_SMD:R_0402_1005Metric, symbol Device:R
- removed SW1: MIC MUTE (DPDT slide), Button_Switch_SMD:SW_DPDT_CK_JS202011JCQN, symbol Switch:SW_DPDT_x2
- added Q6: 2N7002, Package_TO_SOT_SMD:SOT-23, symbol Transistor_FET:2N7002
- C12: value 100nF -> 10uF; footprint Capacitor_SMD:C_0402_1005Metric -> Capacitor_SMD:C_0603_1608Metric
- C13: value 10uF -> 100nF; footprint Capacitor_SMD:C_0603_1608Metric -> Capacitor_SMD:C_0402_1005Metric
- R10: value 10k -> 1M
- R7: value 100k -> 33R
- R9: value 1k -> 10k
Connections:
- net MIC_MUTE_STATUS is gone; now on net GND: R10.2
- net MUTE_LED_A is gone; now on net CM5_3V3: R9.2
- net +5V_CM5: now also C12.1
- net AMP_SD_MODE: now also R10.1
- net GND: now also Q6.2 (S); no longer R7.2
- net I2S_DIN: now also R7.2
- net MIC_SD renamed MIC_DATA_GATED
- net MIC_VDD renamed MIC_SW_LIVE
- net MIC_SW_LIVE: now also Q6.1 (G); no longer C12.1
- net MUTE_LED_PWR renamed MUTE_STATUS_IO
- net MUTE_STATUS_IO: now also Q6.3 (D); no longer R10.1
Other:
- note added: "MAX98357A amp; mic data/mute-status interface to the side-key flex. Connections are by net label at pin endpoints; global labels cross sheets."
- note removed: "Mics (2x SPH0645LM4H), hardware mic mute, MAX98357A amp. Connections are by net label at pin endpoints; global labels cross sheets."
- title: PocketMate - Mics (2x SPH0645LM4H), hardware mic mute, MAX98357A amp -> PocketMate - Audio
