File: hardware/kicad/cm5.kicad_sch (KiCad schematic)
At the start: 12 parts, among them J1 10164227-1001A1RLF, J2 10164227-1001A1RLF

Commit message: Sync KiCad schematic to netlist v3.2; add side_flex sheet
Parts:
- added C7: 1uF, Capacitor_SMD:C_0402_1005Metric, symbol Device:C
- added J12: Fan 5V/GND/PWM/TACH, Connector_JST:JST_SH_SM04B-SRSS-TB_1x04-1MP_P1.00mm_Horizontal, symbol Connector_Generic:Conn_01x04
- added R3: 10k, Resistor_SMD:R_0402_1005Metric, symbol Device:R
- J1: footprint (none) -> PocketMate:CM5_B2B_10164227_Pins1-100
- J2: footprint (none) -> PocketMate:CM5_B2B_10164227_Pins101-200
Connections:
- net +5V_CM5: now also C7.1, J12.1 (Pin_1)
- net CM5_3V3: now also R3.2
- net GND: now also C7.2, J12.2 (Pin_2)
- net FAN_TACH: now reaches J1.16 (Fan_Tacho)
- net FAN_TACH: now also J12.4 (Pin_4), R3.1
- net FAN_PWM: now reaches J1.19 (Fan_PWM)
- net FAN_PWM: now also J12.3 (Pin_3)
- net CSI_D2_N: now reaches J2.133 (MIPI0_D2_N)
- net CSI_D2_P: now reaches J2.135 (MIPI0_D2_P)
- net CSI_D3_N: now reaches J2.139 (MIPI0_D3_N)
- net CSI_D3_P: now reaches J2.141 (MIPI0_D3_P)
- net DSI_D2_N: now reaches J2.193 (MIPI1_D2_N)
- net DSI_D3_N: now reaches J2.194 (MIPI1_D3_N)
- net DSI_D2_P: now reaches J2.195 (MIPI1_D2_P)
- net DSI_D3_P: now reaches J2.196 (MIPI1_D3_P)
- net MIC_MUTE_STATUS renamed MUTE_STATUS_IO
- no-connect marks 102 -> 92
Other:
- title: PocketMate - CM5 module B2B connectors -> PocketMate - CM5

Commit message: Sync schematic with LTE link sheet (lte_link.kicad_sch), generator, nets, ERC report and PDF
Connections:
- net LTE_W_DISABLE_N: now reaches J1.24 (GPIO26)
- net LTE_RESET: now reaches J1.28 (GPIO13)
- net LTE_STATUS: now reaches J1.29 (GPIO16)
- net LTE_PWRKEY: now reaches J1.30 (GPIO6)
- net LTE_RI: now reaches J1.31 (GPIO12)
- net LTE_PWR_EN: now reaches J1.34 (GPIO5)
- net LTE_AP_READY: now reaches J1.41 (GPIO25)
- net LTE_USB_DP: now reaches J2.134 (USB3-0-DP)
- net LTE_USB_DM: now reaches J2.136 (USB3-0-DM)
- no-connect marks 92 -> 83
Other:
- moved on the sheet: C1, C2, C3, C4, C5, C6, C7, J12, J2, R1, R2, R3
