File: hardware/kicad/mcu.kicad_sch (KiCad schematic)
At the start: 25 parts, among them J8 SWD (TC2030 pads), Q4 2N7002, Q5 2N7002, SW1 POWER, SW2 ACTION, SW3 VOL+, SW4 VOL-, U9 STM32U031K8U6

Commit message: Sync KiCad schematic to netlist v3.2; add side_flex sheet
Parts:
- removed C41, C42: 100nF, Capacitor_SMD:C_0402_1005Metric, symbol Device:C
- removed C43: 1uF, Capacitor_SMD:C_0402_1005Metric, symbol Device:C
- removed Q4, Q5: 2N7002, Package_TO_SOT_SMD:SOT-23, symbol Device:Q_NMOS
- removed R33, R34: 1k, Resistor_SMD:R_0402_1005Metric, symbol Device:R
- removed R35: 10k, Resistor_SMD:R_0402_1005Metric, symbol Device:R
- removed SW1: POWER, Button_Switch_SMD:SW_SPST_PTS810, symbol Switch:SW_Push
- removed SW2: ACTION, Button_Switch_SMD:SW_SPST_PTS810, symbol Switch:SW_Push
- removed SW3: VOL+, Button_Switch_SMD:SW_SPST_PTS810, symbol Switch:SW_Push
- removed SW4: VOL-, Button_Switch_SMD:SW_SPST_PTS810, symbol Switch:SW_Push
- added C49, C50, C51, C52: 10nF, Capacitor_SMD:C_0402_1005Metric, symbol Device:C
- added C53, C54: 100nF, Capacitor_SMD:C_0402_1005Metric, symbol Device:C
- added D5: PESD5V0S1BB (ESD, MIC_SW_LIVE), Diode_SMD:D_SOD-523, symbol Device:D_TVS
- added J10: Skin NTC 10k B3435, Connector_JST:JST_SH_SM02B-SRSS-TB_1x02-1MP_P1.00mm_Horizontal, symbol Connector_Generic:Conn_01x02
- added J11: FH12-16S-0.5SH(55), Connector_FFC-FPC:Hirose_FH12-16S-0.5SH_1x16-1MP_P0.50mm_Horizontal, symbol Connector_Generic:Conn_01x16
- added Q4, Q5: 2N7002, Package_TO_SOT_SMD:SOT-23, symbol Transistor_FET:2N7002
- added R42, R43, R44, R46, R47: 100k, Resistor_SMD:R_0402_1005Metric, symbol Device:R
- added R45: 0R, Resistor_SMD:R_0402_1005Metric, symbol Device:R
- added U13: TPD4E05U06DQAR (flex buttons ESD), Package_SON:USON-10_2.5x1.0mm_P0.5mm, symbol Power_Protection:TPD4E05U06DQA
- added U14: TPS22917DBVR, Package_TO_SOT_SMD:SOT-23-6, symbol Power_Management:TPS22917DBV
- C45, C47, C48: value 10nF -> 100nF
- C46: value 10nF -> 1uF
- R36, R40: value 100k -> 10k
- R37: value 100k -> 10k 1%
- R38, R39: value 100k -> 1k
Connections:
- net +3V3_AON: now also C44.1, C45.1, C46.1, R41.2, J11.2 (Pin_2), R42.2, R43.2, R44.2; no longer R36.2, R37.2, R38.2, R39.2
- net BOOST_EN: now also U9.25 (PA15); no longer U9.14 (PB0)
- net BTN_ACTION_N: now also C50.1, J11.16 (Pin_16), R42.1, U13.2 (D1-); no longer C46.1, R37.1
- net BTN_PWR_N: now also R41.1, C49.1, J11.12 (Pin_12), U13.1 (D1+); no longer C45.1, R36.1
- net BTN_VOLDN_N: now also C52.1, J11.14 (Pin_14), R44.1, U13.5 (D2-); no longer C48.1, R39.1
- net BTN_VOLUP_N: now also C51.1, J11.13 (Pin_13), R43.1, U13.4 (D2+); no longer C47.1, R38.1
- net CM5_3V3: now also R40.2
- net CM5_PMIC_EN: now also Q5.3 (D)
- net CM5_PMIC_OFF_DRV: now also Q5.1 (G), R47.1; no longer R41.1
- net CM5_PWRBTN_DRV: now also Q4.1 (G), R46.1; no longer R40.1
- net CM5_PWR_BUTTON: now also Q4.3 (D)
- net GND: now also R36.2, C49.2, C50.2, C51.2, C52.2, C53.2, C54.2, D5.1 (A1), J10.2 (Pin_2), J11.1 (Pin_1), J11.5 (Pin_5), J11.8 (Pin_8), Q4.2 (S), Q5.2 (S), R46.2, R47.2, U13.3 (GND), U13.8 (GND), U14.2 (GND); no longer R40.2, R41.2
- net MCU_IRQ_N: now also R40.1
- net MCU_NRST: now also C47.1; no longer C44.1
- net MCU_RX: now also R39.1
- net MCU_TX: now also R38.1
- net UART0_RX: now also R38.2
- net UART0_TX: now also R39.2
- net MIC_PWR_EN: now reaches U9.21 (PA11)
- net MIC_PWR_EN: now also U14.3 (ON)
- net NTC_BIAS: now reaches U9.22 (PA12)
- net NTC_BIAS: now also R37.1
- net MCU_BOOT0: now reaches U9.31 (PF3)
- net MCU_BOOT0: now also R36.1
- net MIC_MUTE_STATUS renamed MUTE_STATUS_IO
- net PMIC_SCL renamed MCU_I2C_SCL
- net MCU_I2C_SCL: now also J11.10 (Pin_10)
- net PMIC_SDA renamed MCU_I2C_SDA
- net MCU_I2C_SDA: now also J11.9 (Pin_9)
- new net +3V3_PERIPH: J11.15 (Pin_15)
- new net I2S_BCLK: J11.4 (Pin_4)
- new net I2S_LRCLK: J11.6 (Pin_6)
- new net MICSW_QOD: R45.1, U14.5 (QOD)
- new net MIC_DATA_GATED: J11.7 (Pin_7)
- new net MIC_FEED: C54.1, J11.3 (Pin_3), R45.2, U14.6 (VOUT)
- new net MIC_SW_LIVE: C53.1, D5.2 (A2), J11.11 (Pin_11), U14.1 (VIN)
- new net NTC_ADC: C48.1, J10.1 (Pin_1), R37.2, U9.14 (PB0)
- no-connect marks 6 -> 7
Other:
- title: PocketMate - STM32U031 always-on supervisor, buttons, CM5 power control -> PocketMate - MCU
