File: hardware/kicad/power_input.kicad_sch (KiCad schematic)
At the start: 36 parts, among them J6 USB-C 16P, J7 Battery 1S (BAT+,NTC,BAT-), Q1 PMOS 30V (e.g. SiSS27DN) VERI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, U2 USBLC6-2SC6 (D+/D-), U3 USBLC6-2SC6 (CC1/CC2), U4 STUSB4500QTR, U5 BQ25895RTWR, U6 MAX17055ETB+

Commit message: Sync KiCad schematic to netlist v3.2; add side_flex sheet
Parts:
- removed C26: 470nF, Capacitor_SMD:C_0402_1005Metric, symbol Device:C
- removed J7: Battery 1S (BAT+,NTC,BAT-), Connector_JST:JST_SH_SM03B-SRSS-TB_1x03-1MP_P1.00mm_Horizontal, symbol Connector_Generic:Conn_01x03
- removed Q1: PMOS 30V (e.g. SiSS27DN) VERIFY, Package_TO_SOT_SMD:SOT-23, symbol Device:Q_PMOS
- removed R24: 10k, Resistor_SMD:R_0402_1005Metric, symbol Device:R
- added C14: 1uF, Capacitor_SMD:C_0402_1005Metric, symbol Device:C
- added J7: Molex 205338-0005 (BAT+,BAT+,BAT-,BAT-,NTC), PocketMate:Molex_Pico-Lock_205338-0005_1x05-1MP_P2.00mm_Horizontal, symbol Connector_Generic:Conn_01x05
- added Q1: DMP3013SFV, Package_SON:Diodes_PowerDI3333-8, symbol Transistor_FET:DMP3013SFV
- added R11: 1k, Resistor_SMD:R_0603_1608Metric, symbol Device:R
- added R12: 220R, Resistor_SMD:R_0603_1608Metric, symbol Device:R
- C16: footprint Capacitor_SMD:C_0402_1005Metric -> Capacitor_SMD:C_0603_1608Metric
- C18: value 1uF -> 10uF; footprint Capacitor_SMD:C_0603_1608Metric -> Capacitor_SMD:C_0805_2012Metric
- C19: value 10uF -> 47nF; footprint Capacitor_SMD:C_0805_2012Metric -> Capacitor_SMD:C_0402_1005Metric
- C20: value 47nF -> 4.7uF; footprint Capacitor_SMD:C_0402_1005Metric -> Capacitor_SMD:C_0603_1608Metric
- C21: value 4.7uF -> 22uF; footprint Capacitor_SMD:C_0603_1608Metric -> Capacitor_SMD:C_0805_2012Metric
- C23: value 22uF -> 10uF
- C24: value 10uF -> 100nF; footprint Capacitor_SMD:C_0805_2012Metric -> Capacitor_SMD:C_0402_1005Metric
- C25: value 100nF -> 470nF
- J6: value USB-C 16P -> TYPE-C-31-M-12; footprint Connector_USB:USB_C_Receptacle_GCT_USB4105-xx-A_16P_TopMnt_Horizontal -> Connector_USB:USB_C_Receptacle_HRO_TYPE-C-31-M-12
- L1: value 1uH -> 1uH XAL4020-102ME; footprint Inductor_SMD:L_Taiyo-Yuden_MD-3030 -> Inductor_SMD:L_Coilcraft_XAL4020-XXX
- R13: value 1k -> 100k; footprint Resistor_SMD:R_0603_1608Metric -> Resistor_SMD:R_0402_1005Metric
- R14: value 100k -> 130R 1%
- R15: value 260R -> 5.23k
- R16: value 5.23k -> 30.1k
- R17: value 30.1k -> 2.2k
- R18: value 2.2k -> 10m 1% 1206 0.5W; footprint Resistor_SMD:R_0402_1005Metric -> Resistor_SMD:R_1206_3216Metric
- R19: value 10m 1% 0603 -> 4.7k; footprint Resistor_SMD:R_0603_1608Metric -> Resistor_SMD:R_0402_1005Metric
- R21: value 4.7k -> 10k
- U6: footprint (none) -> PocketMate:Maxim_TDFN-10-1EP_2x2.5mm_P0.4mm_EP1.4x1.3mm_MAX17055
Connections:
- net +3V3_AON: now also R19.2
- net BAT_N: now also C24.2, R18.1, J7.3 (Pin_3), J7.4 (Pin_4); no longer R19.1
- net CHG_BTST: now also C19.1; no longer C20.1
- net CHG_ILIM: now also R14.1; no longer R15.1
- net CHG_INT_N: now also R22.1; no longer R23.1
- net CHG_PMID: now also C18.1; no longer C19.1
- net CHG_REGN: now also C20.1, R15.1, R17.1; no longer C21.1, R16.1, R18.1
- net CHG_STAT_LED_A: now also R17.2; no longer R18.2
- net CHG_SW: now also C19.2; no longer C20.2
- net CHG_TS: now also R15.2, R16.1, J7.5 (Pin_5); no longer R16.2, R17.1
- net GAUGE_ALRT_N: now also R23.1
- net GAUGE_REG: now also C25.1
- net GND: now also C20.2, R14.2, R16.2, R18.2, C14.2; no longer C19.2, C24.2, R15.2, R17.2, R19.2
- net PD_ALERT_N: now also R21.1; no longer R22.1
- net PD_DISCH: now also R12.1; no longer R13.1
- net PD_VREG_1V2: now also C14.1; no longer C15.1
- net PD_VREG_2V7: now also C15.1; no longer C16.1
- net VBAT: now also C23.1, J7.1 (Pin_1), J7.2 (Pin_2); no longer C25.1
- net VBUS_C: now also C16.1, Q1.1 (S), Q1.2 (S), Q1.3 (S), R11.2; no longer C17.1, R14.2, U4.18 (VBUS_VS_DISCH)
- net VBUS_CHG: now also C17.1, Q1.5 (D), R12.2; no longer C18.1
- net VBUS_EN_SNK: now also R13.1, Q1.4 (G); no longer R14.1
- net VSYS: now also C21.1; no longer C23.1
- net PMIC_SCL renamed MCU_I2C_SCL
- net MCU_I2C_SCL: now also R20.1; no longer R21.1
- net PMIC_SDA renamed MCU_I2C_SDA
- net MCU_I2C_SDA: now also R19.1; no longer R20.1
- new net PD_VBUS_VS: R11.1, U4.18 (VBUS_VS_DISCH)
Other:
- title: PocketMate - USB-C, STUSB4500 PD sink, BQ25895 charger, MAX17055 gauge, battery -> PocketMate - PowerInput
