File: hardware/kicad/regulators.kicad_sch (KiCad schematic)
At the start: 27 parts, among them Q2 PMOS 20V <=10mOhm (e.g. SiSS2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, Q3 2N7002, U7 TPS7A0233PDQNR, U8 TPS61088RHLR

Commit message: Sync KiCad schematic to netlist v3.2; add side_flex sheet
Parts:
- removed Q2: PMOS 20V <=10mOhm (e.g. SiSS23DN) VERIFY, Package_TO_SOT_SMD:SOT-23, symbol Device:Q_PMOS
- removed Q3: 2N7002, Package_TO_SOT_SMD:SOT-23, symbol Device:Q_NMOS
- removed U7: TPS7A0233PDQNR, Package_SON:Texas_X2SON-4_1x1mm_P0.65mm, symbol PocketMate:TPS7A0233PDQN
- added C26: 1uF, Capacitor_SMD:C_0402_1005Metric, symbol Device:C
- added C41, C42: 22uF, Capacitor_SMD:C_0805_2012Metric, symbol Device:C
- added C43: 10nF, Capacitor_SMD:C_0402_1005Metric, symbol Device:C
- added L3: 1uH DFE252012F-1R0M, Inductor_SMD:L_1008_2520Metric, symbol Device:L
- added Q2: DMP3013SFV, Package_SON:Diodes_PowerDI3333-8, symbol Transistor_FET:DMP3013SFV
- added Q3: 2N7002, Package_TO_SOT_SMD:SOT-23, symbol Transistor_FET:2N7002
- added R24: 150k 1%, Resistor_SMD:R_0402_1005Metric, symbol Device:R
- added R33, R34, R35: 100k, Resistor_SMD:R_0402_1005Metric, symbol Device:R
- added U12: TLV62585DRLR, Package_TO_SOT_SMD:SOT-563, symbol PocketMate:TLV62585DRL
- added U7: TPS7A0233PDBVR, Package_TO_SOT_SMD:SOT-23-5, symbol PocketMate:TPS7A0233PDBV
- C28: value 1uF -> 100nF
- C29: value 100nF -> 22uF; footprint Capacitor_SMD:C_0402_1005Metric -> Capacitor_SMD:C_0805_2012Metric
- C30: value 22uF -> 100nF; footprint Capacitor_SMD:C_0805_2012Metric -> Capacitor_SMD:C_0402_1005Metric
- C31: value 100nF -> 2.2uF; footprint Capacitor_SMD:C_0402_1005Metric -> Capacitor_SMD:C_0603_1608Metric
- C32: value 2.2uF -> 100nF; footprint Capacitor_SMD:C_0603_1608Metric -> Capacitor_SMD:C_0402_1005Metric
- C33: value 100nF -> 47nF
- C34: value 47nF -> 2.7nF
- C35: value 2.7nF -> 18pF
- C36: value 22pF -> 22uF; footprint Capacitor_SMD:C_0402_1005Metric -> Capacitor_SMD:C_0805_2012Metric
- C39: value 22uF -> 10uF; footprint Capacitor_SMD:C_0805_2012Metric -> Capacitor_SMD:C_0603_1608Metric
- C40: value 10nF -> 100nF
- L2: value 1.0uH 12A Isat -> 1uH XAL5030-102ME; footprint Inductor_SMD:L_Bourns_SRP5030T -> Inductor_SMD:L_Coilcraft_XAL5030-XXX
- R25: value 301k -> 127k 1%
- R26: value 100k -> 182k 1%
- R27: value 324k 1% -> 56k 1%
- R28: value 100k 1% -> 10k
- R29: value 56k -> 100k
- R30: value 100k -> 100k 1%
- R31: value 100k -> 22.1k 1%
- R32: value 100k -> 10k
- U8: footprint (none) -> PocketMate:TI_RHL0020A_VQFN-20_3.5x4.5mm_TPS61088
Connections:
- net +3V3_AON: now also C27.1, U7.5 (OUT); no longer C29.1
- net +5V_BOOST: now also C36.1, R26.1, C43.2, Q2.1 (S), Q2.2 (S), Q2.3 (S), R34.2; no longer C39.1, C40.2, R27.1, R31.2
- net +5V_CM5: now also Q2.5 (D)
- net BOOST_EN: now also R29.1; no longer R30.1
- net BST_BOOT: now also C32.1; no longer C33.1
- net BST_COMP: now also C35.1, R28.1; no longer C36.1, R29.1
- net BST_COMP_RC: now also C34.1, R28.2; no longer C35.1, R29.2
- net BST_FB: now also R26.2, R27.1; no longer R27.2, R28.1
- net BST_FSW: now also R24.1; no longer R25.1
- net BST_ILIM: now also R25.1; no longer R26.1
- net BST_SS: now also C33.1; no longer C34.1
- net BST_SW: now also C32.2, R24.2; no longer C33.2, R25.2
- net BST_VCC: now also C31.1; no longer C32.1
- net CM5_5V_EN: now also Q3.1 (G), R35.1; no longer R32.1
- net GND: now also C33.2, C40.2, R25.2, R27.2, R29.2, R31.2, C26.2, C41.2, C42.2, Q3.2 (S), R33.2, R35.2, U12.1 (GND), U7.2 (GND); no longer C32.2, R26.2, R28.2, R30.2, R32.2
- net LSW_GATE: now also C43.1, Q2.4 (G), Q3.3 (D), R34.1; no longer C40.1, R31.1
- net VBAT: now also C26.1, U7.1 (IN), U7.3 (EN); no longer C27.1
- net VSYS: now also C29.1, C39.1, C40.1, U12.3 (VIN); no longer C31.1
- new net +3V3_PERIPH: C41.1, C42.1, L3.2, R30.1
- new net BUCK3V3_EN: R32.2, R33.1, U12.4 (EN)
- new net BUCK3V3_FB: R30.2, R31.1, U12.5 (FB)
- new net BUCK3V3_SW: L3.1, U12.2 (SW)
- new net CM5_3V3: R32.1
- no-connect marks 1 -> 3
Other:
- title: PocketMate - Always-on LDO, TPS61088 5V boost, CM5 5V load switch -> PocketMate - Regulators
